File: Card/Card.kicad_pcb (KiCad board)
At the start: 2 copper layers, 85 x 55 mm, 7 parts, among them U1 NT3H2111W0FTTJ

Commit message: Front Side Decorations
Parts:
- added G***: LOGO, LOGO, F.Cu at (137.8, 108.8)
- added G***: LOGO, LOGO, F.Cu at (170.1, 86.1)
- added G*** (x2): LOGO, LOGO, F.Cu at (106.0, 73.5)
- added G***: LOGO, LOGO, F.Cu at (142.0, 87.0)
- added G***: LOGO, LOGO, F.Cu at (152.5, 104.9)
- added G*** (x2): LOGO, LOGO, F.Cu at (140.8, 98.6)
- added G***: LOGO, LOGO, F.Cu at (151.0, 92.0)
- added G***: LOGO, LOGO, F.Cu at (181.1, 110.5)
- added G***: LOGO, LOGO, F.Cu at (143.6, 73.5)
- added G***: LOGO, LOGO, F.Cu at (175.2, 110.6)
Routing:
- net VCC: track 116.5 -> 117.1 mm
Other:
- board text added: "Dynix7"
- board text added: "Embedded Systems & Software Engineer"

Commit message: Backside
Parts:
- added REF**: SOT-23-5, Package_TO_SOT_SMD:SOT-23-5, B.Cu at (137.5, 97.3)
- added REF**: 1206, Resistor_SMD:R_1206_3216Metric, B.Cu at (179.1, 75.3)
- added REF**: SOT-23-8, Package_TO_SOT_SMD:SOT-23-8, B.Cu at (137.5, 102.9)
- added REF**: 0402, Resistor_SMD:R_0402_1005Metric, B.Cu at (179.1, 69.1)
- added REF**: 0603, Resistor_SMD:R_0603_1608Metric, B.Cu at (179.1, 70.8)
- added REF**: SOT-23-3, Package_TO_SOT_SMD:SOT-23-3, B.Cu at (144.0, 97.3)
- added REF**: SOT-223-6, Package_TO_SOT_SMD:SOT-223-6, B.Cu at (154.1, 93.5)
- added REF**: VFBGA-100_7.0x7.0mm_Layout10x10_P0.65mm, Package_BGA:VFBGA-100_7.0x7.0mm_Layout10x10_P0.65mm, B.Cu at (124.0, 102.5)
- added REF**: SOT-223-5, Package_TO_SOT_SMD:SOT-223-5, B.Cu at (165.1, 102.5)
- added REF**: TO-252-2, Package_TO_SOT_SMD:TO-252-2, B.Cu at (158.9, 75.0)
- added REF**: 123, Diode_SMD:D_SOD-123, B.Cu at (168.5, 87.0)
- added REF**: TO-252-3_TabPin2, Package_TO_SOT_SMD:TO-252-3_TabPin2, B.Cu at (158.9, 83.5)
- added REF**: QFN-32, Package_DFN_QFN:QFN-32-1EP_4x4mm_P0.4mm_EP2.65x2.65mm, B.Cu at (117.2, 85.8)
- added REF**: SOT-223-8, Package_TO_SOT_SMD:SOT-223-8, B.Cu at (153.6, 102.5)
- added REF**: TSSOP-16_4.4x5mm_P0.65mm, Package_SO:TSSOP-16_4.4x5mm_P0.65mm, B.Cu at (147.5, 84.0)
- added REF**: TSSOP-8_4.4x3mm_P0.65mm, Package_SO:TSSOP-8_4.4x3mm_P0.65mm, B.Cu at (147.5, 74.5)
- added REF**: 882, Diode_SMD:D_SOD-882, B.Cu at (168.7, 76.0)
- added REF**: Microchip_TFBGA-196_11x11mm_Layout14x14_P0.75mm_SMD, Package_BGA:Microchip_TFBGA-196_11x11mm_Layout14x14_P0.75mm_SMD, B.Cu at (112.1, 97.6)
- added REF**: SOIC-16_3.9x9.9mm_P1.27mm, Package_SO:SOIC-16_3.9x9.9mm_P1.27mm, B.Cu at (138.6, 84.7)
- added REF**: 323, Diode_SMD:D_SOD-323, B.Cu at (168.6, 83.0)
- added REF**: 2512, Resistor_SMD:R_2512_6332Metric, B.Cu at (179.0, 100.5)
- added REF**: QFN-16, Package_DFN_QFN:QFN-16-1EP_3x3mm_P0.5mm_EP1.75x1.75mm, B.Cu at (107.6, 86.3)
- added REF**: 1812, Capacitor_SMD:C_1812_4532Metric, B.Cu at (179.0, 82.2)
- added REF**: 2010, Resistor_SMD:R_2010_5025Metric, B.Cu at (179.1, 89.8)
- added REF**: 2920, Fuse:Fuse_2920_7451Metric, B.Cu at (179.0, 106.1)
- added REF**: 1210, Resistor_SMD:R_1210_3225Metric, B.Cu at (179.1, 78.3)
- added REF**: SOT-23-6, Package_TO_SOT_SMD:SOT-23-6, B.Cu at (144.0, 102.9)
- added REF**: 2220, Capacitor_SMD:C_2220_5750Metric, B.Cu at (179.1, 95.1)
- added REF**: 0805, Resistor_SMD:R_0805_2012Metric, B.Cu at (179.1, 72.8)
- added REF**: ST_UFBGA-81_5x5mm_Layout9x9_P0.5mm, Package_BGA:ST_UFBGA-81_5x5mm_Layout9x9_P0.5mm, B.Cu at (124.0, 94.0)
- added REF**: LQFP-48, Package_QFP:LQFP-48_7x7mm_P0.5mm, B.Cu at (125.5, 74.3)
- added REF**: SOT-223, Package_TO_SOT_SMD:SOT-223, B.Cu at (165.0, 93.5)
- added REF**: QFN-48, Package_DFN_QFN:QFN-48-1EP_5x5mm_P0.35mm_EP3.7x3.7mm, B.Cu at (127.2, 85.7)
- added REF**: 923, Diode_SMD:D_SOD-923, B.Cu at (168.8, 73.0)
- added REF**: SOIC-8_3.9x4.9mm_P1.27mm, Package_SO:SOIC-8_3.9x4.9mm_P1.27mm, B.Cu at (138.6, 74.3)
- added REF**: 1808, Capacitor_SMD:C_1808_4520Metric, B.Cu at (179.0, 86.1)
- added REF**: TQFP-32, Package_QFP:TQFP-32_7x7mm_P0.8mm, B.Cu at (109.6, 74.2)
- added REF**: 523, Diode_SMD:D_SOD-523, B.Cu at (168.6, 79.5)
- added R_0201: 0201, Resistor_SMD:R_0201_0603Metric, B.Cu at (179.1, 67.7)
Routing:
- net (no net): track 0.00 -> 618.6 mm
- net VCC: track 117.1 -> 112.5 mm
- net GND: track 103.4 -> 101.3 mm
Other:
- board text added: "1"
- board text added: "1/10in"
- board text added: "2"
- board text added: "3"
- board text added: "4"
- board text added: "5"
- board text added: "6"
- board text added: "7"
- board text added: "8"
- board text added: "SOD"
- board text added: "SOIC"
- board text added: "SOT-223"
- board text added: "SOT-23"
- board text added: "TO-25"
- board text added: "TSSOP"
- board text added: "cm"
